File: stm32_stick.kicad_pcb (KiCad board)
At the start: 4 copper layers, 20.3 x 63.5 mm, 56 parts, among them J1 FTSH-105-01-F-DV-007-K, J2 Conn_01x20, J3 629105150521, J4 Conn_01x20, J5 Conn_01x05, J6 Conn_01x05, U1 STM32F405RGTx, U2 AMS1117-3.3, U3 USBLC6-2P6, Y1 8MHz

Commit message: boot0 resistro
Parts:
- removed the REF** at (34.4, 106.9)
- added R2: 10k, Resistor_SMD:R_0402_1005Metric, F.Cu at (33.9, 107.8)
- added REF**: via-0.6, via:via-0.6, F.Cu at (46.4, 93.0)
- added REF**: via-0.6, via:via-0.6, F.Cu at (35.7, 89.0)
- added REF**: via-0.6, via:via-0.6, F.Cu at (34.3, 90.4)
- moved REF** 1.97 mm to (43.8, 108.8)
Connections:
- C5 pad 1: Net-(C5-Pad1) -> +5V
- C6 pad 1: Net-(C5-Pad1) -> +5V
- J3 pad 1: Net-(C5-Pad1) -> +5V
- J4 pad 2: +3V3 -> +5V
- U2 pad 3: Net-(C5-Pad1) -> +5V
- U3 pad 5: Net-(C5-Pad1) -> +5V
Routing:
- net +5V: track 0.00 -> 28.9 mm, vias 0 -> 2
- net Net-(C5-Pad1): track 18.8 -> 0.00 mm, vias 2 -> 0
- net BOOT0: track 31.6 -> 35.1 mm
- added copper zone on B.Cu, net GND
Other:
- board text added: "5v"

Commit message: note
Other:
- board text added: "hello from seattle"

Commit message: production outputs
Parts:
- removed the REF** at (39.6, 63.1)
- removed the REF** at (39.1, 61.8)
- added REF**: via-0.6, via:via-0.6, F.Cu at (40.9, 79.9)
- added REF**: via-0.6, via:via-0.6, F.Cu at (40.8, 68.3)
- added REF**: via-0.6, via:via-0.6, F.Cu at (37.3, 69.6)
- added REF**: via-0.6, via:via-0.6, F.Cu at (37.2, 63.5)
- added REF**: via-0.6, via:via-0.6, F.Cu at (40.3, 63.4)
- U3: value USBLC6-2P6 -> USBLC6-2SC6; footprint Package_TO_SOT_SMD:SOT-666 -> Package_TO_SOT_SMD:SOT-23-6
- moved REF** 5.60 mm to (41.9, 64.8)
- moved D1 1.91 mm to (39.4, 70.5)
- moved R1 1.91 mm to (39.4, 72.4)
- moved U3 1.42 mm to (38.7, 66.0)
Routing:
- net +5V: track 28.9 -> 30.6 mm
- net /USB_D+: track 32.4 -> 31.0 mm
