File: stm32_stick.sch (KiCad schematic (older format))
At the start: 21 parts, among them J1 FTSH-105-01-F-DV-007-K, J2 Conn_01x20, J3 629105150521, J4 Conn_01x20, J5 Conn_01x05, J6 Conn_01x05, U1 STM32F405RGTx, U2 AMS1117-3.3, U3 USBLC6-2P6, Y1 8MHz

Commit message: boot0 resistro
Parts:
- added R?: 10k, Resistor_SMD:R_0402_1005Metric, symbol Device:R
- J5, J6: LCSC (none) -> N/A
Connections:
- net +3V3: no longer J4.2 (Pin_2)
- net BOOT0: now also R?.1
- net GND: now also R?.2
- net +5V: now reaches C5.1, C6.1, J3.1 (VBUS), U2.3 (VI), U3.5 (VBUS)
- net +5V: now also J4.2 (Pin_2)
Changed lines of the file:
@@
 	0    -1   -1   0
-$EndComp
-$Comp
-L power:+3.3V #PWR0118
-U 1 1 5F5F8B85
-P 9975 2975
-F 0 "#PWR0118" H 9975 2825 50  0001 C CNN
-F 1 "+3.3V" V 9990 3103 50  0000 L CNN
-F 2 "" H 9975 2975 50  0001 C CNN
-F 3 "" H 9975 2975 50  0001 C CNN
-	1    9975 2975
-	0    1    1    0
 $EndComp
 Text GLabel 3250 5400 2    50   Input ~ 0
@@
 F 2 "Connector_PinHeader_2.54mm:PinHeader_1x05_P2.54mm_Vertical" H 8075 5100 50  0001 C CNN
 F 3 "~" H 8075 5100 50  0001 C CNN
+F 4 "N/A" H 8075 5100 50  0001 C CNN "LCSC"
 	1    8075 5100
 	-1   0    0    -1
@@
 F 2 "Connector_PinHeader_2.54mm:PinHeader_1x05_P2.54mm_Vertical" H 9775 5075 50  0001 C CNN
 F 3 "~" H 9775 5075 50  0001 C CNN
+F 4 "N/A" H 9775 5075 50  0001 C CNN "LCSC"
 	1    9775 5075
 	-1   0    0    -1
@@
 Wire Wire Line
 	9975 5275 10075 5275
-Text GLabel 1550 4100 0    50   Input ~ 0
+Text GLabel 850  4100 0    50   Input ~ 0
 BOOT0
 Wire Wire Line
-	1550 4100 1750 4100
+	850  4100 950  4100
 Text GLabel 8400 5300 2    50   Input ~ 0
 BOOT0
 Wire Wire Line
 	8400 5300 8275 5300
+$Comp
+L power:+5V #PWR0118
+U 1 1 5F5AA783
+P 9975 2975
+F 0 "#PWR0118" H 9975 2825 50  0001 C CNN
+F 1 "+5V" V 9990 3103 50  0000 L CNN
+F 2 "" H 9975 2975 50  0001 C CNN
+F 3 "" H 9975 2975 50  0001 C CNN
+	1    9975 2975
+	0    1    1    0
+$EndComp
+$Comp
+L power:+5V #PWR0125
+U 1 1 5F5ABE0F
+P 3750 1000
+F 0 "#PWR0125" H 3750 850 50  0001 C CNN
+F 1 "+5V" H 3765 1173 50  0000 C CNN
+F 2 "" H 3750 1000 50  0001 C CNN
+F 3 "" H 3750 1000 50  0001 C CNN
+	1    3750 1000
+	1    0    0    -1
+$EndComp
+$Comp
+L Device:R R?
+U 1 1 5F5BC576
+P 950 4300
+F 0 "R?" H 1020 4346 50  0000 L CNN
+F 1 "10k" H 1020 4255 50  0000 L CNN
+F 2 "Resistor_SMD:R_0402_1005Metric" V 880 4300 50  0001 C CNN
+F 3 "~" H 950 4300 50  0001 C CNN
+F 4 "C25744" H 950 4300 50  0001 C CNN "LCSC"
+	1    950  4300
+	1    0    0    -1
+$EndComp
+$Comp
+L power:GND #PWR?
+U 1 1 5F5BC5E1
+P 950 4450
+F 0 "#PWR?" H 950 4200 50  0001 C CNN
+F 1 "GND" H 955 4277 50  0000 C CNN
+F 2 "" H 950 4450 50  0001 C CNN
+F 3 "" H 950 4450 50  0001 C CNN
+	1    950  4450
+	1    0    0    -1
+$EndComp
+Wire Wire Line
+	950  4150 950  4100
+Connection ~ 950  4100
+Wire Wire Line
+	950  4100 1750 4100
 $EndSCHEMATC

Commit message: note
Parts:
- gave numbers to parts that had none: 1
Changed lines of the file:
@@
 $EndComp
 $Comp
-L Device:R R?
+L Device:R R2
 U 1 1 5F5BC576
 P 950 4300
-F 0 "R?" H 1020 4346 50  0000 L CNN
+F 0 "R2" H 1020 4346 50  0000 L CNN
 F 1 "10k" H 1020 4255 50  0000 L CNN
 F 2 "Resistor_SMD:R_0402_1005Metric" V 880 4300 50  0001 C CNN
@@
 $EndComp
 $Comp
-L power:GND #PWR?
+L power:GND #PWR0126
 U 1 1 5F5BC5E1
 P 950 4450
-F 0 "#PWR?" H 950 4200 50  0001 C CNN
+F 0 "#PWR0126" H 950 4200 50  0001 C CNN
 F 1 "GND" H 955 4277 50  0000 C CNN
 F 2 "" H 950 4450 50  0001 C CNN

Commit message: production outputs
Parts:
- removed U3: USBLC6-2P6, Package_TO_SOT_SMD:SOT-666, symbol Power_Protection:USBLC6-2P6
- added U3: USBLC6-2SC6, Package_TO_SOT_SMD:SOT-23-6, symbol Power_Protection:USBLC6-2SC6
Connections:
- net +5V: now also U3.5 (VBUS)
- net GND: now also U3.2 (GND)
- net USB_D+: now also U3.1 (IO1), U3.6 (IO1)
- net USB_D-: now also U3.3 (IO2), U3.4 (IO2)
Other:
- moved on the sheet: C8, C9
Changed lines of the file:
@@
 	10075 5175 9975 5175
-$Comp
-L Power_Protection:USBLC6-2P6 U3
-U 1 1 5F7F214E
-P 3750 2050
-F 0 "U3" H 3900 1700 50  0000 C CNN
-F 1 "USBLC6-2P6" H 3400 1675 50  0000 C CNN
-F 2 "Package_TO_SOT_SMD:SOT-666" H 3750 1550 50  0001 C CNN
-F 3 "https://www.st.com/resource/en/datasheet/usblc6-2.pdf" H 3950 2400 50  0001 C CNN
-F 4 "C7519" H 3750 2050 50  0001 C CNN "LCSC"
-	1    3750 2050
-	1    0    0    -1
-$EndComp
 $Comp
 L power:GND #PWR0119
 U 1 1 5F7F49BC
-P 3750 2450
-F 0 "#PWR0119" H 3750 2200 50  0001 C CNN
-F 1 "GND" H 3755 2277 50  0000 C CNN
-F 2 "" H 3750 2450 50  0001 C CNN
-F 3 "" H 3750 2450 50  0001 C CNN
-	1    3750 2450
+P 3750 2650
+F 0 "#PWR0119" H 3750 2400 50  0001 C CNN
+F 1 "GND" H 3755 2477 50  0000 C CNN
+F 2 "" H 3750 2650 50  0001 C CNN
+F 3 "" H 3750 2650 50  0001 C CNN
+	1    3750 2650
 	1    0    0    -1
 $EndComp
@@
 Wire Wire Line
 	3750 1000 3975 1000
-Text Label 3275 2050 2    50   ~ 0
+Text Label 3175 2150 2    50   ~ 0
 USB_D+
-Text Label 4225 2050 0    50   ~ 0
-USB_D-
-Wire Wire Line
-	4225 1950 4150 1950
-Wire Wire Line
-	4225 2150 4150 2150
-Wire Wire Line
-	4225 1950 4225 2150
-Wire Wire Line
-	3350 2150 3275 2150
-Wire Wire Line
-	3275 2150 3275 1950
-Wire Wire Line
-	3275 1950 3350 1950
+Wire Wire Line
+	3250 2250 3175 2250
+Wire Wire Line
+	3175 2250 3175 2050
+Wire Wire Line
+	3175 2050 3250 2050
 $Comp
 L Device:LED D1
@@
 L Device:C C8
 U 1 1 5F861B89
-P 3150 3300
-F 0 "C8" H 3265 3346 50  0000 L CNN
-F 1 "100n" H 3265 3255 50  0000 L CNN
-F 2 "Capacitor_SMD:C_0402_1005Metric" H 3188 3150 50  0001 C CNN
-F 3 "~" H 3150 3300 50  0001 C CNN
-F 4 "C1525" H 3150 3300 50  0001 C CNN "LCSC"
-	1    3150 3300
+P 875 3275
+F 0 "C8" H 990 3321 50  0000 L CNN
+F 1 "100n" H 990 3230 50  0000 L CNN
+F 2 "Capacitor_SMD:C_0402_1005Metric" H 913 3125 50  0001 C CNN
+F 3 "~" H 875 3275 50  0001 C CNN
+F 4 "C1525" H 875 3275 50  0001 C CNN "LCSC"
+	1    875  3275
 	1    0    0    -1
 $EndComp
@@
 L power:GND #PWR0121
 U 1 1 5F862106
-P 3150 3450
-F 0 "#PWR0121" H 3150 3200 50  0001 C CNN
-F 1 "GND" H 3155 3277 50  0000 C CNN
-F 2 "" H 3150 3450 50  0001 C CNN
-F 3 "" H 3150 3450 50  0001 C CNN
-	1    3150 3450
+P 875 3425
+F 0 "#PWR0121" H 875 3175 50  0001 C CNN
+F 1 "GND" H 880 3252 50  0000 C CNN
+F 2 "" H 875 3425 50  0001 C CNN
+F 3 "" H 875 3425 50  0001 C CNN
+	1    875  3425
 	1    0    0    -1
 $EndComp
@@
 L power:+3.3V #PWR0122
 U 1 1 5F862A25
-P 3150 3150
-F 0 "#PWR0122" H 3150 3000 50  0001 C CNN
-F 1 "+3.3V" H 3165 3323 50  0000 C CNN
-F 2 "" H 3150 3150 50  0001 C CNN
-F 3 "" H 3150 3150 50  0001 C CNN
-	1    3150 3150
+P 875 3125
+F 0 "#PWR0122" H 875 2975 50  0001 C CNN
+F 1 "+3.3V" H 890 3298 50  0000 C CNN
+F 2 "" H 875 3125 50  0001 C CNN
+F 3 "" H 875 3125 50  0001 C CNN
+	1    875  3125
 	1    0    0    -1
 $EndComp
@@
 L Device:C C9
 U 1 1 5F862D86
-P 3575 3300
-F 0 "C9" H 3690 3346 50  0000 L CNN
-F 1 "100n" H 3690 3255 50  0000 L CNN
-F 2 "Capacitor_SMD:C_0402_1005Metric" H 3613 3150 50  0001 C CNN
-F 3 "~" H 3575 3300 50  0001 C CNN
-F 4 "C1525" H 3575 3300 50  0001 C CNN "LCSC"
-	1    3575 3300
+P 1300 3275
+F 0 "C9" H 1415 3321 50  0000 L CNN
+F 1 "100n" H 1415 3230 50  0000 L CNN
+F 2 "Capacitor_SMD:C_0402_1005Metric" H 1338 3125 50  0001 C CNN
+F 3 "~" H 1300 3275 50  0001 C CNN
+F 4 "C1525" H 1300 3275 50  0001 C CNN "LCSC"
+	1    1300 3275
 	1    0    0    -1
 $EndComp
@@
 L power:GND #PWR0123
 U 1 1 5F8632E2
-P 3575 3450
-F 0 "#PWR0123" H 3575 3200 50  0001 C CNN
-F 1 "GND" H 3580 3277 50  0000 C CNN
-F 2 "" H 3575 3450 50  0001 C CNN
-F 3 "" H 3575 3450 50  0001 C CNN
-	1    3575 3450
+P 1300 3425
+F 0 "#PWR0123" H 1300 3175 50  0001 C CNN
+F 1 "GND" H 1305 3252 50  0000 C CNN
+F 2 "" H 1300 3425 50  0001 C CNN
+F 3 "" H 1300 3425 50  0001 C CNN
+	1    1300 3425
 	1    0    0    -1
 $EndComp
@@
 L power:+3.3V #PWR0124
 U 1 1 5F8636BC
-P 3575 3150
-F 0 "#PWR0124" H 3575 3000 50  0001 C CNN
-F 1 "+3.3V" H 3590 3323 50  0000 C CNN
-F 2 "" H 3575 3150 50  0001 C CNN
-F 3 "" H 3575 3150 50  0001 C CNN
-	1    3575 3150
+P 1300 3125
+F 0 "#PWR0124" H 1300 2975 50  0001 C CNN
+F 1 "+3.3V" H 1315 3298 50  0000 C CNN
+F 2 "" H 1300 3125 50  0001 C CNN
+F 3 "" H 1300 3125 50  0001 C CNN
+	1    1300 3125
 	1    0    0    -1
 $EndComp
@@
 Wire Wire Line
 	950  4100 1750 4100
+$Comp
+L Power_Protection:USBLC6-2SC6 U3
+U 1 1 5F83C7B4
+P 3750 2150
+F 0 "U3" H 3750 2831 50  0000 C CNN
+F 1 "USBLC6-2SC6" H 3750 2740 50  0000 C CNN
+F 2 "Package_TO_SOT_SMD:SOT-23-6" H 3000 2550 50  0001 C CNN
+F 3 "http://www2.st.com/resource/en/datasheet/CD00050750.pdf" H 3950 2500 50  0001 C CNN
+	1    3750 2150
+	1    0    0    -1
+$EndComp
+Wire Wire Line
+	4325 2050 4325 2250
+Wire Wire Line
+	4325 2250 4250 2250
+Wire Wire Line
+	4325 2050 4250 2050
+Text Label 4325 2150 0    50   ~ 0
+USB_D-
 $EndSCHEMATC
